Commit message: add additional ee link and ee heading task: using qua vs using joint angle directly

File: resources/robots/cassie/urdf/cassie.urdf (robot description, URDF)
Before this commit: robot cassie, 16 links, 15 joints
Links:
- added link iiwa_link1, mass 0.1627406257303; visual mesh filename=../meshes/iiwa_link1.STL scale=1.0 1.0 1.0
Joints:
- added joint iiwa_joint1: type revolute, parent base, child iiwa_link1, origin xyz=0 0 0.333 rpy=0 0 0, axis 0 0 1, limit lower=-2.9671 upper=2.9671 effort=10 velocity=2.1750
