Commit message: test wheeled base rl training

File: resources/robots/s1_base/urdf/astribot_s1_base.urdf (robot description, URDF)
Before this commit: robot astribot_s1_base, 85 links, 84 joints
Links:
- link astribot_torso_base: geometry collision cylinder length=0.18 radius=0.27; visual mesh filename=../mesh/torso_v3/Base_T_simple.STL
Joints:
- joint wheel_LF_Joint: limit lower=-3.14159 upper=3.14159 effort=300 velocity=100 -> lower=-3.14159 upper=3.14159 effort=50 velocity=100
- joint wheel_LR_Joint: limit lower=-3.14159 upper=3.14159 effort=300 velocity=100 -> lower=-3.14159 upper=3.14159 effort=50 velocity=100
- joint wheel_RF_Joint: limit lower=-3.14159 upper=3.14159 effort=300 velocity=100 -> lower=-3.14159 upper=3.14159 effort=50 velocity=100
- joint wheel_RR_Joint: limit lower=-3.14159 upper=3.14159 effort=300 velocity=100 -> lower=-3.14159 upper=3.14159 effort=50 velocity=100

Commit message: add collision filter for rollers only

File: resources/robots/s1_base/urdf/astribot_s1_base.urdf (robot description, URDF)
Before this commit: robot astribot_s1_base, 85 links, 84 joints
Joints:
- joint wheel_LF_Joint: limit lower=-3.14159 upper=3.14159 effort=50 velocity=100 -> lower=-3.14159 upper=3.14159 effort=100 velocity=100
- joint wheel_LR_Joint: limit lower=-3.14159 upper=3.14159 effort=50 velocity=100 -> lower=-3.14159 upper=3.14159 effort=100 velocity=100
- joint wheel_RF_Joint: limit lower=-3.14159 upper=3.14159 effort=50 velocity=100 -> lower=-3.14159 upper=3.14159 effort=100 velocity=100
- joint wheel_RR_Joint: limit lower=-3.14159 upper=3.14159 effort=50 velocity=100 -> lower=-3.14159 upper=3.14159 effort=100 velocity=100

Commit message: fix bug: training fail 1. bigger terrian herizontal/vertical scale 2. larger map 1 is to reduce collision buffer stress 2 is to avoid falling at map edge, which causing value fn loss error

File: resources/robots/s1_base/urdf/astribot_s1_base.urdf (robot description, URDF)
Before this commit: robot astribot_s1_base, 85 links, 84 joints
Joints:
- joint wheel_LF_Joint: limit lower=-3.14159 upper=3.14159 effort=100 velocity=100 -> lower=-3.14159 upper=3.14159 effort=20 velocity=25
- joint wheel_LR_Joint: limit lower=-3.14159 upper=3.14159 effort=100 velocity=100 -> lower=-3.14159 upper=3.14159 effort=20 velocity=25
- joint wheel_RF_Joint: limit lower=-3.14159 upper=3.14159 effort=100 velocity=100 -> lower=-3.14159 upper=3.14159 effort=20 velocity=25
- joint wheel_RR_Joint: limit lower=-3.14159 upper=3.14159 effort=100 velocity=100 -> lower=-3.14159 upper=3.14159 effort=20 velocity=25
